Commit message: Consume the IMU: driver, description, broadcaster, and an on-robot EKF
The firmware has served IMU data for a long time (`i`), and SerialMcu can
parse it, but nothing ever called it. This wires it through:

- andino_base: honour `baud_rate` (it was hardcoded to 57600 with a TODO);
  read encoders and IMU in ONE exchange when the description declares an IMU
  <sensor> and the firmware reports one; export the ten state interfaces
  imu_sensor_broadcaster claims. A unit-norm check on the quaternion doubles
  as an integrity check of the whole line: a truncated or timed-out reply
  parses as zeros, and is now discarded instead of teleporting both wheels
  back to tick zero.
- andino_description: the <sensor>, an `imu_link`, 115200 baud, and a serial
  timeout of 100 ms instead of a full second (one lost reply used to stall the
  control loop for 50 cycles).
- andino_control: imu_sensor_broadcaster defined (spawned only by launch
  files that want it) with static covariances, and honest covariances on the
  wheel odometry so a downstream filter lets the gyro outvote wheel yaw.
- andino_bringup: robot_base.launch.py spawns the broadcaster (-> `imu/data`)
  and hands odom -> base_link to the new robot_ekf.launch.py, which fuses
  wheel velocities with the gyro's yaw rate. The fused ORIENTATION is left out
  on purpose for now — NDOF mode steers heading by a magnetometer that sits
  next to two DC motors; see config/ekf.yaml.

Upstream's single-process bringup is untouched: it keeps the controller's own
odom TF and does not spawn the broadcaster.

Co-Authored-By: Claude Fable 5.1 <noreply@anthropic.com>
Claude-Session: https://claude.ai/code/session_0185YSDjcU9pDPxNpMumMVfv

File: andino_description/urdf/andino.urdf.xacro (robot description, xacro)
@@ -78,4 +78,14 @@
   <xacro:camera_sensor parent_link="base_link" sensor_prop="${sensor_prop}">
   </xacro:camera_sensor>
+  <!-- IMU (BNO055, read through the microcontroller). Yaw fusion is indifferent to where on the
+       chassis the sensor sits, so the offset is left at zero; the ROTATION is what matters. It
+       assumes the board lies flat, component side up. Check it on the robot, upright: turned
+       counter-clockwise seen from above, the yaw reported in this frame must increase. -->
+  <link name="imu_link"/>
+  <joint name="imu_joint" type="fixed">
+    <parent link="base_link"/>
+    <child link="imu_link"/>
+    <origin xyz="0 0 0" rpy="0 0 0"/>
+  </joint>
   <!-- ros2_control -->
   <xacro:if value="$(arg use_real_ros_control)">

File: andino_description/urdf/include/andino_control.urdf.xacro (robot description, xacro)
@@ -33,4 +33,19 @@
         <state_interface name="position"/>
       </joint>
+      <!-- The BNO055 on the microcontroller's I2C bus. The driver reads it in the same serial
+           exchange as the encoders, and only if the firmware reports one (`h`). These ten are what
+           imu_sensor_broadcaster claims. -->
+      <sensor name="imu_sensor">
+        <state_interface name="orientation.x"/>
+        <state_interface name="orientation.y"/>
+        <state_interface name="orientation.z"/>
+        <state_interface name="orientation.w"/>
+        <state_interface name="angular_velocity.x"/>
+        <state_interface name="angular_velocity.y"/>
+        <state_interface name="angular_velocity.z"/>
+        <state_interface name="linear_acceleration.x"/>
+        <state_interface name="linear_acceleration.y"/>
+        <state_interface name="linear_acceleration.z"/>
+      </sensor>
     </ros2_control>
   </xacro:macro>
